File: hardware/bike_pov.sch (KiCad schematic (older format))
At the start: 1 part

Commit message: ughhh
Parts:
- removed LD?: LDO_ TC1014-2.7VCT713, symbol LDO_~TC1014-2.7VCT713
- added D1, D10, D100, D101, D102, D103, D104, D105, D106, D107, D108, D109, D11, D110, D111, D112, D113, D114, D115, D116, D117, D118, D119, D12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: RGB_LED, symbol RGB_LED
- added U? (x4): TLC590, symbol TLC590
Connections:
- net labels added: BLANK, DCPRG, GSCLK, SCLK, SIN, VCC, VPRG, XERR, XLAT
- net labels removed: Bypass, SHUD, VIN, VOUT
- wire segments 0 -> 150
